File: placa/polarización/placa-polarizacion.kicad_pcb (KiCad board)
At the start: 2 copper layers, 19 parts, among them P1 CONN_01X03, P2 CONN_01X03, Q1 2N7002, Q2 IRLML5203PbF, SW1 Switch_SPDT_x2, U1 LM324

Commit message: Revision de la placa
Parts:
- moved P1 16.3 mm to (70.4, 45.2), turned to 180 degrees
- moved P2 15.3 mm to (93.3, 35.0)
- moved C5 8.54 mm to (94.9, 39.2), turned to 0 degrees
- moved R2 3.17 mm to (73.4, 75.6)
- moved SW1 2.61 mm to (109.0, 63.9)
- moved R4 1.75 mm to (94.0, 65.9)
- moved C3 0.26 mm to (91.8, 45.2)
Routing:
- net GND: track 34.8 -> 85.1 mm
- net /iON: track 98.8 -> 60.1 mm
- net VDD: track 59.1 -> 79.9 mm
- net VSS: track 91.1 -> 107.3 mm
- net Net-(C5-Pad1): track 25.6 -> 31.5 mm
- net /i50: track 50.9 -> 53.3 mm
- net Net-(RV2-Pad2): track 27.1 -> 29.0 mm
- net Net-(C5-Pad2): track 33.5 -> 31.7 mm
- net Net-(Q2-Pad2): track 11.0 -> 9.43 mm
- net Net-(Q1-Pad2): track 16.3 -> 14.9 mm
- net Net-(RV1-Pad2): track 31.5 -> 32.1 mm
- added copper zone on B.Cu, net GND
Other:
- board outline added: 52.4 x 53.3 mm
- board text added: "Medidas 2 RF-SWITCH Polarización"
